File: MacroPAD/MacroPad_PCB/MacroPAD/_autosave-MacroPAD.kicad_sch (KiCad schematic)
At the start: 59 parts, among them J2 AVR-ISP-6, SW1 SW_Push, SW2 RotaryEncoder, U1 ATmega32U4-A, U2 USB6B1, Y1 16MHz

Commit message: MacroPAD V0.3: Added additional filter for rotary encoder for debounce purpose
Parts:
- R10, R11: footprint Resistor_SMD:R_1206_3216Metric -> Resistor_SMD:R_0603_1608Metric
Other:
- note added: "Mounting holes"
- moved on the sheet: H1, H2, H3, H4
Changed lines of the file:
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@@
 	)
 	(junction
-		(at 135.89 130.81)
+		(at 132.08 134.62)
 		(diameter 0)
 		(color 0 0 0 0)
@@
 	)
 	(junction
-		(at 127 130.81)
+		(at 123.19 134.62)
 		(diameter 0)
 		(color 0 0 0 0)
 	)
 	(junction
-		(at 144.78 130.81)
+		(at 140.97 134.62)
 		(diameter 0)
 		(color 0 0 0 0)
@@
 	(wire
 		(pts
-			(xy 118.11 130.81) (xy 127 130.81)
+			(xy 114.3 134.62) (xy 123.19 134.62)
 		)
 		(stroke
@@
 		)
 	)
+	(polyline
+		(pts
+			(xy 176.53 123.19) (xy 176.53 124.46)
+		)
+		(stroke
+			(width 0)
+			(type dash)
+		)
+	)
 	(wire
 		(pts
@@
 	(polyline
 		(pts
-			(xy 128.27 117.475) (xy 128.27 86.36)
+			(xy 128.27 122.555) (xy 128.27 86.36)
 		)
 		(stroke
@@
 		)
 	)
+	(polyline
+		(pts
+			(xy 176.53 142.24) (xy 176.53 124.46)
+		)
+		(stroke
+			(width 0)
+			(type dash)
+		)
+	)
 	(wire
 		(pts
@@
 	(wire
 		(pts
-			(xy 135.89 130.81) (xy 144.78 130.81)
+			(xy 132.08 134.62) (xy 140.97 134.62)
 		)
 		(stroke
@@
 	(wire
 		(pts
-			(xy 127 130.81) (xy 135.89 130.81)
+			(xy 123.19 134.62) (xy 132.08 134.62)
 		)
 		(stroke
@@
 		)
 	)
+	(text "Mounting holes"
+		(exclude_from_sim no)
+		(at 97.282 125.476 0)
+		(effects
+			(font
+				(size 1.27 1.27)
+			)
+		)
+	)
 	(text "LED strip (x6)"
 		(exclude_from_sim no)
@@
 	(symbol
 		(lib_id "Mechanical:MountingHole_Pad")
-		(at 144.78 128.27 0)
+		(at 140.97 132.08 0)
 		(unit 1)
 		(exclude_from_sim yes)
@@
 		(fields_autoplaced yes)
 		(property "Reference" "H4"
-			(at 147.32 125.7299 0)
+			(at 143.51 129.5399 0)
 			(effects
 				(font
@@
 		)
 		(property "Value" "M4"
-			(at 147.32 128.2699 0)
+			(at 143.51 132.0799 0)
 			(effects
 				(font
@@
 		)
 		(property "Footprint" "MountingHole:MountingHole_3.2mm_M3_Pad_Via"
-			(at 144.78 128.27 0)
+			(at 140.97 132.08 0)
 			(effects
 				(font
@@
 		)
 		(property "Datasheet" "~"
-			(at 144.78 128.27 0)
+			(at 140.97 132.08 0)
 			(effects
 				(font
@@
 		)
 		(property "Description" "Mounting Hole with connection"
-			(at 144.78 128.27 0)
+			(at 140.97 132.08 0)
 			(effects
 				(font
@@
 	(symbol
 		(lib_id "Mechanical:MountingHole_Pad")
-		(at 118.11 128.27 0)
+		(at 114.3 132.08 0)
 		(unit 1)
 		(exclude_from_sim yes)
@@
 		(fields_autoplaced yes)
 		(property "Reference" "H1"
-			(at 120.65 125.7299 0)
+			(at 116.84 129.5399 0)
 			(effects
 				(font
@@
 		)
 		(property "Value" "M1"
-			(at 120.65 128.2699 0)
+			(at 116.84 132.0799 0)
 			(effects
 				(font
@@
 		)
 		(property "Footprint" "MountingHole:MountingHole_3.2mm_M3_Pad_Via"
-			(at 118.11 128.27 0)
+			(at 114.3 132.08 0)
 			(effects
 				(font
@@
 		)
 		(property "Datasheet" "~"
-			(at 118.11 128.27 0)
+			(at 114.3 132.08 0)
 			(effects
 				(font
@@
 		)
 		(property "Description" "Mounting Hole with connection"
-			(at 118.11 128.27 0)
+			(at 114.3 132.08 0)
 			(effects
 				(font
@@
 	(symbol
 		(lib_id "Mechanical:MountingHole_Pad")
-		(at 135.89 128.27 0)
+		(at 132.08 132.08 0)
 		(unit 1)
 		(exclude_from_sim yes)
@@
 		(fields_autoplaced yes)
 		(property "Reference" "H3"
-			(at 138.43 125.7299 0)
+			(at 134.62 129.5399 0)
 			(effects
 				(font
@@
 		)
 		(property "Value" "M3"
-			(at 138.43 128.2699 0)
+			(at 134.62 132.0799 0)
 			(effects
 				(font
@@
 		)
 		(property "Footprint" "MountingHole:MountingHole_3.2mm_M3_Pad_Via"
-			(at 135.89 128.27 0)
+			(at 132.08 132.08 0)
 			(effects
 				(font
@@
 		)
 		(property "Datasheet" "~"
-			(at 135.89 128.27 0)
+			(at 132.08 132.08 0)
 			(effects
 				(font
@@
 		)
 		(property "Description" "Mounting Hole with connection"
-			(at 135.89 128.27 0)
+			(at 132.08 132.08 0)
 			(effects
 				(font
@@
 	(symbol
 		(lib_id "Mechanical:MountingHole_Pad")
-		(at 127 128.27 0)
+		(at 123.19 132.08 0)
 		(unit 1)
 		(exclude_from_sim yes)
@@
 		(fields_autoplaced yes)
 		(property "Reference" "H2"
-			(at 129.54 125.7299 0)
+			(at 125.73 129.5399 0)
 			(effects
 				(font
@@
 		)
 		(property "Value" "M2"
-			(at 129.54 128.2699 0)
+			(at 125.73 132.0799 0)
 			(effects
 				(font
@@
 		)
 		(property "Footprint" "MountingHole:MountingHole_3.2mm_M3_Pad_Via"
-			(at 127 128.27 0)
+			(at 123.19 132.08 0)
 			(effects
 				(font
@@
 		)
 		(property "Datasheet" "~"
-			(at 127 128.27 0)
+			(at 123.19 132.08 0)
 			(effects
 				(font
@@
 		)
 		(property "Description" "Mounting Hole with connection"
-			(at 127 128.27 0)
+			(at 123.19 132.08 0)
 			(effects
 				(font
@@
 	(symbol
 		(lib_id "power:GND")
-		(at 144.78 130.81 0)
+		(at 140.97 134.62 0)
 		(unit 1)
 		(exclude_from_sim no)
@@
 		(dnp no)
 		(property "Reference" "#PWR025"
-			(at 144.78 137.16 0)
+			(at 140.97 140.97 0)
 			(effects
 				(font
@@
 		)
 		(property "Value" "GND"
-			(at 144.78 134.366 0)
+			(at 140.97 138.176 0)
 			(effects
 				(font
@@
 		)
 		(property "Footprint" ""
-			(at 144.78 130.81 0)
+			(at 140.97 134.62 0)
 			(effects
 				(font
@@
 		)
 		(property "Datasheet" ""
-			(at 144.78 130.81 0)
+			(at 140.97 134.62 0)
 			(effects
 				(font
@@
 		)
 		(property "Description" "Power symbol creates a global label with name \"GND\" , ground"
-			(at 144.78 130.81 0)
+			(at 140.97 134.62 0)
 			(effects
 				(font
@@
 			)
 		)
-		(property "Footprint" "Resistor_SMD:R_1206_3216Metric"
+		(property "Footprint" "Resistor_SMD:R_0603_1608Metric"
 			(at 107.95 100.33 0)
 			(effects
@@
 			)
 		)
-		(property "Footprint" "Resistor_SMD:R_1206_3216Metric"
+		(property "Footprint" "Resistor_SMD:R_0603_1608Metric"
 			(at 107.95 110.49 0)
 			(effects
