File: MacroPAD/MacroPad_PCB/MacroPAD/MacroPAD.kicad_sch (KiCad schematic)
At the start: 59 parts, among them J2 AVR-ISP-6, SW1 SW_Push, SW2 RotaryEncoder, U1 ATmega32U4-A, U2 USB6B1, Y1 16MHz

Commit message: Added MPN for the BOM
Parts:
- C1, C2, C3: MPN (none) -> C0603C104K5RACTU
- C10, C7, C8, C9: MPN (none) -> C0603C106M8PACTU
- C11, C12: MPN (none) -> C0603C103K5RACTU
- C4: MPN (none) -> CL10A105KB8NNNC
- C5, C6: MPN (none) -> CL10C120JB8NNNC
- D1, D2, D3, D4, D5, D6: MPN (none) -> 1N4148W-13-F
- D10, D11, D12, D13: MPN (none) -> COM-16347
- D14: MPN (none) -> LG R971-KN-1-0-20-R18
- D15: MPN (none) -> LTST-C150YKT
- D16: MPN (none) -> LTST-C150KRKT
- J2: MPN (none) -> 61200621621
- R1: MPN (none) -> RC1206FR-0710KL
- R1-C1, R1-C2, R1-C3, R2-C1, R2-C2, R2-C3, R3-C1, R3-C2, R3-C3: MPN (none) -> PG151101S11
- R10, R11: footprint Resistor_SMD:R_1206_3216Metric -> Resistor_SMD:R_0603_1608Metric; MPN (none) -> RC0603FR-0710KL
- R2, R3: MPN (none) -> RC0603FR-0722RL
- R4, R5: MPN (none) -> CR0603-FX-5101ELF
- R6: MPN (none) -> RC0603FR-0710KL
- R7: value 1k -> 220; MPN (none) -> CRGCQ0805F220R
- R8, R9: value 1k -> 220; MPN (none) -> CRG1206F220R
- SW1: MPN (none) -> SKHHAKA010
- SW2: MPN (none) -> PEC12R-4225F-N0024
- U1: MPN (none) -> ATmega32U4-A
- U2: MPN (none) -> USB6B1
- USB-C1: MPN (none) -> 2171790001
- Y1: MPN (none) -> ECS-160-20-33-TR
Other:
- note added: "Mounting holes"
- moved on the sheet: H1, H2, H3, H4
